File: PCB/main/procon_gcc_main_pcb.kicad_pcb (KiCad board)
At the start: 4 copper layers, 110.9 x 59.7 mm, 130 parts, among them J1 Conn_01x04_Pin, J3 To Button Board, J5 Conn_01x02_Pin, J9 USB_C_Receptacle, Q1 Q_PMOS_GDS, Q2 Q_NMOS_GSD, Q3 Q_NMOS_GSD, Q4 BSS138DW, Q5 BSS138DW, Q7 MMBT3904, Q8 MMBT3904, SW1 GL18_SW, SW2 GL18_SW, SW3 1TS026A-1000-0550, SW4 TS35CA, SW5 1TS026A-1000-0550, T1 36-8730, T2 36-8730, T3 36-8730, T4 36-8730, U1 GH39F (Hall SOT23), U10 MCP3002, U11 ST_LSM6, U12 PI3USB4000A, U13 GD25Q80EEIGR, U14 TPS630001RCR, U16 BQ25180, U2 GH39F (Hall SOT23), U3 GH39F (Hall SOT23), U4 GH39F (Hall SOT23), U5 ST_LSM6, U6 RP2040, U7 CH340K, U8 MCP3002, U9 ESP32-PICO-MINI-02, Y1 Crystal_GND3

Commit message: haptic test build
Parts:
- removed D1: M7C, Diode_SMD:D_SOD-123
- removed F1: Fuse, Fuse:Fuse_1206_3216Metric_Pad1.42x1.75mm_HandSolder
- removed Q1: Q_PMOS_GDS, Package_TO_SOT_SMD:SOT-23
- removed Q2, Q3: Q_NMOS_GSD, Package_TO_SOT_SMD:SOT-23
- removed R1: 10k, Resistor_SMD:R_0201_0603Metric
- removed R2: 100R, Resistor_SMD:R_0201_0603Metric
- removed TP5: TestPoint, TestPoint:TestPoint_Pad_D1.5mm
- added C30: 1uF, Capacitor_SMD:C_0201_0603Metric, F.Cu at (162.2, 117.2)
- added C31: 1uF, Capacitor_SMD:C_0201_0603Metric, F.Cu at (159.7, 121.9)
- added C32: 100n, Capacitor_SMD:C_0201_0603Metric, F.Cu at (153.9, 114.8)
- added C33: 1uF, Capacitor_SMD:C_0201_0603Metric, F.Cu at (165.7, 117.2)
- added C34: 1uF, Capacitor_SMD:C_0201_0603Metric, F.Cu at (163.8, 121.9)
- added R37: 1.2k, Resistor_SMD:R_0201_0603Metric, F.Cu at (153.1, 114.8)
- added R38: 1k, Resistor_SMD:R_0201_0603Metric, F.Cu at (164.6, 117.5)
- added U15: DRV2605LYZFR, Package_BGA:Texas_DSBGA-9_1.4715x1.4715mm_Layout3x3_P0.5mm, F.Cu at (160.7, 119.7)
- added U17: PI5A3157CEX, Package_TO_SOT_SMD:SOT-363_SC-70-6, F.Cu at (155.9, 113.0)
- added U18: DRV2605LYZFR, Package_BGA:Texas_DSBGA-9_1.4715x1.4715mm_Layout3x3_P0.5mm, F.Cu at (164.2, 119.7)
- R3: value 10k -> 1k
- R4: value 100R -> 1k
- SW1, SW2: footprint progcc_v3:GL18 -> hhl:GL18
- SW4: footprint progcc_v3:TS35CA -> hhl:TS35CA
- U1, U2, U3, U4: footprint progcc_v3:GH39F -> hhl:GH39F
- moved R4 8.31 mm to (161.0, 117.5), turned to 0 degrees
- moved R5 6.18 mm to (158.6, 118.9), turned to 90 degrees
- moved R3 3.51 mm to (151.9, 114.4), turned to 180 degrees
Connections:
- R3 pad 1: GND -> LRA_FILTERED
- R3 pad 2: R_BRAKE -> LRA_IN
- R4 pad 1: RUMBLE -> LRA_SDA_1
- R4 pad 2: Net-(Q3-G) -> +3V3
- R5 pad 1: GND -> Net-(U15-EN)
- R5 pad 2: RUMBLE -> +3V3
- T1 pad 1: VBUS_SYS -> LRA2_OUT_-
- T2 pad 1: RUMBLE- -> LRA1_OUT_+
- T3 pad 1: VBUS_SYS -> LRA1_OUT_-
- T4 pad 1: RUMBLE- -> LRA2_OUT_+
- U6 pad 36: RUMBLE -> LRA_IN
- U6 pad 37: R_BRAKE -> LRA_SDA_SELECT
Routing:
- net VBUS_SYS: track 172.7 -> 27.1 mm, vias 6 -> 4
- net RUMBLE-: track 127.3 -> 0.00 mm, vias 4 -> 0
- net LRA1_OUT_+: track 0.00 -> 91.4 mm, vias 0 -> 4
- net LRA1_OUT_-: track 0.00 -> 90.0 mm, vias 0 -> 1
- net LRA2_OUT_-: track 0.00 -> 37.9 mm, vias 0 -> 1
- net LRA2_OUT_+: track 0.00 -> 35.1 mm
- net I2C_SCL: track 39.0 -> 57.6 mm, vias 3 -> 5
- net LRA_FILTERED: track 0.00 -> 18.4 mm, vias 0 -> 2
- net RUMBLE: track 18.2 -> 0.00 mm
- net +3V3: track 88.3 -> 103.6 mm, vias 38 -> 44
- net R_BRAKE: track 13.5 -> 0.00 mm
- net LRA_SDA_2: track 0.00 -> 13.4 mm, vias 0 -> 2
- net LRA_SDA_SELECT: track 0.00 -> 13.0 mm
- net LRA_SDA_1: track 0.00 -> 11.3 mm
- net LRA_IN: track 0.00 -> 9.62 mm
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