File: PCB/main/procon_gcc_main_pcb.kicad_sch (KiCad schematic)
At the start: 124 parts, among them J1 Conn_01x04_Pin, J3 To Button Board, J5 Conn_01x02_Pin, J9 USB_C_Receptacle, Q1 Q_PMOS_GDS, Q2 Q_NMOS_GSD, Q3 Q_NMOS_GSD, Q4 BSS138DW, Q5 BSS138DW, Q7 MMBT3904, Q8 MMBT3904, SW1 1TS026A-1000-0550, SW1 GL18_SW, SW2 GL18_SW, SW4 TS35CA, T1 36-8730, T2 36-8730, T3 36-8730, T4 36-8730, U1 GH39F (Hall SOT23), U10 MCP3002, U11 ST_LSM6, U12 PI3USB4000A, U16 BQ25180, U2 GD25Q80EEIGR, U2 GH39F (Hall SOT23), U3 GH39F (Hall SOT23), U4 GH39F (Hall SOT23), U4 TPS630001RCR, U5 ST_LSM6, U6 RP2040, U7 CH340K, U8 MCP3002, U9 ESP32-PICO-MINI-02, Y1 Crystal_GND3

Commit message: haptic test build
Parts:
- removed D1: M7C, Diode_SMD:D_SOD-123, symbol Device:D_Schottky
- removed F1: Fuse, Fuse:Fuse_1206_3216Metric_Pad1.42x1.75mm_HandSolder, symbol Device:Fuse
- removed Q1: Q_PMOS_GDS, Package_TO_SOT_SMD:SOT-23, symbol Device:Q_PMOS_GSD
- removed Q2, Q3: Q_NMOS_GSD, Package_TO_SOT_SMD:SOT-23, symbol Device:Q_NMOS_GSD
- removed R1: 10k, Resistor_SMD:R_0201_0603Metric, symbol Device:R
- removed R2: 100R, Resistor_SMD:R_0201_0603Metric, symbol Device:R
- removed TP5: TestPoint, TestPoint:TestPoint_Pad_D1.5mm, symbol Connector:TestPoint
- added C24 (x4): 1uF, Capacitor_SMD:C_0201_0603Metric, symbol Device:C
- added C24: 100n, Capacitor_SMD:C_0201_0603Metric, symbol Device:C
- added R37: 1.2k, Resistor_SMD:R_0201_0603Metric, symbol Device:R
- added R38: 1k, Resistor_SMD:R_0201_0603Metric, symbol Device:R
- added U15, U18: DRV2605LYZFR, Package_BGA:Texas_DSBGA-9_1.4715x1.4715mm_Layout3x3_P0.5mm, symbol hhl:DRV2605LYZFR
- added U17: PI5A3157CEX, Package_TO_SOT_SMD:SOT-363_SC-70-6, symbol hhl:PI5A3157CEX
- R3: value 10k -> 1k; LCSC C25804 -> (none)
- R4: value 100R -> 1k; LCSC C22775 -> (none)
- R5: LCSC C25804 -> (none)
- SW1, SW2: footprint progcc_v3:GL18 -> hhl:GL18
- SW4: footprint progcc_v3:TS35CA -> hhl:TS35CA
- U1, U2, U3, U4: footprint progcc_v3:GH39F -> hhl:GH39F
Connections:
- net +3V3: now also R4.2, R5.2, C24.1, C24.1, R38.2, U15.C2 (VDD), U17.5 (VDD), U18.C2 (VDD)
- net GND: now also C24.1, C24.1, C24.1, C24.2, C24.2, R37.1, U15.B3 (GND), U17.2 (GND), U18.B3 (GND); no longer R3.1, R5.1
- net I2C_SCL: now also U15.C1 (SCL), U18.C1 (SCL)
- net I2C_SDA: now also U17.4 (A)
- net VBUS_SYS: no longer T1.1, T3.1
- removed net RUMBLE: R4.1, R5.2, U6.36 (GPIO24)
- net RUMBLE- renamed LRA1_OUT_+
- net LRA1_OUT_+: now also U15.A3 (OUT+); no longer T4.1
- net R_BRAKE renamed LRA_IN
- net LRA_IN: now also U6.36 (GPIO24); no longer U6.37 (GPIO25)
- new net: C24.2, U15.A2 (REG)
- new net: R5.1, U15.A1 (EN), U18.A1 (EN)
- new net: C24.2, U18.A2 (REG)
- new net LRA1_OUT_-: T3.1, U15.C3 (OUT-)
- new net LRA2_OUT_+: T4.1, U18.A3 (OUT+)
- new net LRA2_OUT_-: T1.1, U18.C3 (OUT-)
- new net LRA_FILTERED: C24.2, R3.1, R37.2, U15.B1 (IN/TRIG), U18.B1 (IN/TRIG)
- new net LRA_SDA_1: R4.1, U15.B2 (SDA), U17.3 (B0)
- new net LRA_SDA_2: R38.1, U17.1 (B1), U18.B2 (SDA)
- new net LRA_SDA_SELECT: U17.6 (SEL), U6.37 (GPIO25)
Other:
- note removed: "RUMBLE+"
- company: HHL/Esca -> HHL
- title: ProGCC v3 Main Board -> ProGCC v3+ Main Board
- moved on the sheet: T1, T4
