File: PCB/main_haptic/procon_gcc_main_pcb.kicad_pcb (KiCad board)
At the start: 4 copper layers, 110.9 x 59.7 mm, 132 parts, among them J1 Conn_01x04_Pin, J3 To Button Board, J5 Conn_01x02_Pin, J9 USB_C_Receptacle, Q4 BSS138DW, Q5 BSS138DW, Q7 MMBT3904, Q8 MMBT3904, SW1 GL18_SW, SW2 GL18_SW, SW3 1TS026A-1000-0550, SW4 TS35CA, SW5 1TS026A-1000-0550, T1 36-8730, T2 36-8730, T3 36-8730, T4 36-8730, U1 GH39F (Hall SOT23), U10 MCP3002, U11 ST_LSM6, U12 PI3USB4000A, U13 GD25Q80EEIGR, U14 TPS630001RCR, U15 DRV2605LYZFR, U16 BQ25180, U17 PI5A3157CEX, U18 DRV2605LYZFR, U2 GH39F (Hall SOT23), U3 GH39F (Hall SOT23), U4 GH39F (Hall SOT23), U5 ST_LSM6, U6 RP2040, U7 CH340K, U8 MCP3002, U9 ESP32-PICO-MINI-02, Y1 Crystal_GND3

Commit message: Update hardware layout etc.
Parts:
- removed C33, C34: 1uF, Capacitor_SMD:C_0201_0603Metric
- removed U17: PI5A3157CEX, Package_TO_SOT_SMD:SOT-363_SC-70-6
- removed U18: DRV2605LYZFR, Package_BGA:Texas_DSBGA-9_1.4715x1.4715mm_Layout3x3_P0.5mm
- added J2: SM02B-SURS-TF_LF__SN_, hhl:JST_SM02B-SURS-TF_LF__SN_, F.Cu at (96.0, 144.2)
- added J4: SM02B-SURS-TF_LF__SN_, hhl:JST_SM02B-SURS-TF_LF__SN_, F.Cu at (180.7, 144.1)
- added R1: 0R, Resistor_SMD:R_0603_1608Metric_Pad0.98x0.95mm_HandSolder, F.Cu at (143.9, 105.9)
- added R2: 0R, Resistor_SMD:R_0603_1608Metric_Pad0.98x0.95mm_HandSolder, F.Cu at (142.3, 105.9)
- R38, R4: value 1k -> 0R; footprint Resistor_SMD:R_0201_0603Metric -> Resistor_SMD:R_0603_1608Metric_Pad0.98x0.95mm_HandSolder
- moved R38 9.77 mm to (156.4, 112.1)
- moved T1 7.50 mm to (178.5, 139.9), turned to 0 degrees
- moved T4 7.40 mm to (183.0, 139.9), turned to 0 degrees
- moved R4 6.01 mm to (156.4, 113.7)
- moved T3 5.06 mm to (94.4, 134.9), turned to -90 degrees
- moved T2 3.17 mm to (94.4, 138.9), turned to -90 degrees
- moved J3 3.05 mm to (103.0, 145.3)
- moved D2 1.27 mm to (152.4, 106.7)
- moved F2 1.27 mm to (147.8, 106.5)
- moved C16 1.27 mm to (152.7, 104.6)
- moved C32 0.71 mm to (153.3, 114.3)
- moved R3 0.71 mm to (151.4, 114.0)
- moved R37 0.71 mm to (152.6, 114.3)
- moved TP4 0.33 mm to (146.9, 102.6)
- moved C25 0.22 mm to (164.3, 110.8)
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Connections:
- R3 pad 2: LRA_IN -> LRA_IN_HI
- R38 pad 1: LRA_SDA_2 -> VBUS_PRE
- R38 pad 2: +3V3 -> VBUS_SYS
- R4 pad 1: LRA_SDA_1 -> VBUS_PRE
- R4 pad 2: +3V3 -> VBUS_SYS
- T1 pad 1: LRA2_OUT_- -> LRA_OUT_-
- T2 pad 1: LRA1_OUT_+ -> LRA_OUT_+
- T3 pad 1: LRA1_OUT_- -> LRA_OUT_-
- T4 pad 1: LRA2_OUT_+ -> LRA_OUT_+
- U15 pad A3: LRA1_OUT_+ -> LRA_OUT_+
- U15 pad B2: LRA_SDA_1 -> I2C_SDA
- U15 pad C3: LRA1_OUT_- -> LRA_OUT_-
- U6 pad 32: IMU1_CS -> LRA_IN_HI
- U6 pad 36: LRA_IN -> LRA_IN_HI
- U6 pad 37: LRA_SDA_SELECT -> IMU1_CS
Routing:
- net LRA_OUT_-: track 0.00 -> 136.2 mm, vias 0 -> 2
- net LRA_OUT_+: track 0.00 -> 134.1 mm, vias 0 -> 5
- net LRA1_OUT_+: track 91.4 -> 0.00 mm, vias 4 -> 0
- net LRA1_OUT_-: track 90.0 -> 0.00 mm, vias 1 -> 0
- net LRA2_OUT_-: track 37.9 -> 0.00 mm, vias 1 -> 0
- net LRA2_OUT_+: track 35.1 -> 0.00 mm
- net VBUS_PRE: track 27.1 -> 44.9 mm, vias 1 -> 3
- net LRA_SDA_2: track 13.4 -> 0.00 mm, vias 2 -> 0
- net LRA_SDA_SELECT: track 13.0 -> 0.00 mm
- net LRA_IN_HI: track 0.00 -> 12.7 mm
- net LRA_SDA_1: track 11.3 -> 0.00 mm
- net I2C_SDA: track 45.3 -> 56.5 mm
- net +3V3: track 103.6 -> 93.7 mm, vias 44 -> 40
- net LRA_IN: track 9.62 -> 0.00 mm
- net Net-(U15-EN): track 8.75 -> 1.65 mm, vias 2 -> 0
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Other:
- board text added: "ProGCC 3.1"
- board text removed: "Additional Design Work: Phob Team"
- board text removed: "ProGCC 3+"
