File: PCB/main_haptic/procon_gcc_main_pcb.kicad_sch (KiCad schematic)
At the start: 126 parts, among them J1 Conn_01x04_Pin, J3 To Button Board, J5 Conn_01x02_Pin, J9 USB_C_Receptacle, Q4 BSS138DW, Q5 BSS138DW, Q7 MMBT3904, Q8 MMBT3904, SW1 1TS026A-1000-0550, SW1 GL18_SW, SW2 GL18_SW, SW4 TS35CA, T1 36-8730, T2 36-8730, T3 36-8730, T4 36-8730, U1 GH39F (Hall SOT23), U10 MCP3002, U11 ST_LSM6, U12 PI3USB4000A, U15 DRV2605LYZFR, U16 BQ25180, U17 PI5A3157CEX, U18 DRV2605LYZFR, U2 GD25Q80EEIGR, U2 GH39F (Hall SOT23), U3 GH39F (Hall SOT23), U4 GH39F (Hall SOT23), U4 TPS630001RCR, U5 ST_LSM6, U6 RP2040, U7 CH340K, U8 MCP3002, U9 ESP32-PICO-MINI-02, Y1 Crystal_GND3

Commit message: Update hardware layout etc.
Parts:
- removed C24 (x2): 1uF, Capacitor_SMD:C_0201_0603Metric, symbol Device:C
- removed U17: PI5A3157CEX, Package_TO_SOT_SMD:SOT-363_SC-70-6, symbol hhl:PI5A3157CEX
- removed U18: DRV2605LYZFR, Package_BGA:Texas_DSBGA-9_1.4715x1.4715mm_Layout3x3_P0.5mm, symbol hhl:DRV2605LYZFR
- added J2, J4: SM02B-SURS-TF_LF__SN_, hhl:JST_SM02B-SURS-TF_LF__SN_, symbol hhl:SM02B-SURS-TF_LF__SN_
- added R1, R2: 0R, Resistor_SMD:R_0603_1608Metric_Pad0.98x0.95mm_HandSolder, symbol Device:R
- R38, R4: value 1k -> 0R; footprint Resistor_SMD:R_0201_0603Metric -> Resistor_SMD:R_0603_1608Metric_Pad0.98x0.95mm_HandSolder
Connections:
- net LRA2_OUT_+ is gone; now on net LRA_OUT_+: T4.1
- net LRA2_OUT_- is gone; now on net LRA_OUT_-: T1.1
- net LRA_SDA_2 is gone; now on net VBUS_PRE: R38.1
- net LRA_SDA_SELECT is gone; now on net IMU1_CS: U6.37 (GPIO25)
- net +3V3: no longer R38.2, R4.2
- net D+: now also R2.1
- net D-: now also R1.1
- net GND: now also J2.S1 (SHIELD), J2.S2 (SHIELD), J4.S1 (SHIELD), J4.S2 (SHIELD)
- net I2C_SDA: now also U15.B2 (SDA)
- net IMU1_CS: no longer U6.32 (GPIO21)
- net RP_USB+: now also R2.2
- net RP_USB-: now also R1.2
- net VBUS_PRE: now also R4.1
- net VBUS_SYS: now also R38.2, R4.2
- net LRA1_OUT_+ renamed LRA_OUT_+
- net LRA_OUT_+: now also J2.2, J4.2
- net LRA1_OUT_- renamed LRA_OUT_-
- net LRA_OUT_-: now also J2.1, J4.1
- net LRA_IN renamed LRA_IN_HI
- net LRA_IN_HI: now also U6.32 (GPIO21)
- removed net LRA_SDA_1: R4.1, U15.B2 (SDA)
Other:
- note added: "PWM2 B"
- note added: "PWM4 A"
- note added: "USB Direct Bypass"
- moved on the sheet: C24, R3, R37, R5, U15
