File: PCB/main_3.2/progcc_3.2_main.kicad_sch (KiCad schematic)
At the start: 136 parts, among them J1 Conn_01x04_Pin, J2 SM02B-SURS-TF_LF__SN_, J3 To Button Board, J4 SM02B-SURS-TF_LF__SN_, J5 Conn_01x02_Pin, J9 USB_C_Receptacle, Q1 MMBT2222A, Q2 MMBT2222A, Q4 BSS138DW, Q5 BSS138DW, Q7 MMBT3904, Q8 MMBT3904, SW1 1TS026A-1000-0550, SW1 GL1807SYAE-002, SW2 GL1807SYAE-002, SW4 TS35CA, T1 36-8730, T2 36-8730, T3 36-8730, T4 36-8730, U10 MCP3002, U11 ST_LSM6, U12 PI3USB4000A, U16 BQ25180, U2 GD25Q80EEIGR, U4 TPS63001DRCR, U5 ST_LSM6, U6 RP2040, U7 CH340K, U8 MCP3002, U9 ESP32-PICO-MINI-02, Y1 Crystal_GND3

Commit message: Update PCB Files
- Standardize differing resistor sizes
- Update oscillator
Parts:
- removed R19: 1k, Resistor_SMD:R_0201_0603Metric, symbol Device:R_Small
- removed Y1: Crystal_GND3, Crystal:Resonator_SMD_Murata_CSTxExxV-3Pin_3.0x1.1mm, symbol Device:Crystal_GND3
- added C35, C36: 15pF, Capacitor_SMD:C_0402_1005Metric, symbol Device:C
- added R19: 1k, Resistor_SMD:R_0201_0603Metric, symbol Device:R
- added Y1: ABM8-272-T3, Crystal:Crystal_SMD_3225-4Pin_3.2x2.5mm, symbol Device:Crystal_GND24
- C1: value 47uF 6.3v -> 47uF; LCSC (none) -> C7190; MPN (none) -> CC0603JRX7R9BB473; Price (none) -> 0.0544
- C10, C11, C12, C9: value .047u -> 47nF; footprint Capacitor_SMD:C_0603_1608Metric_Pad1.08x0.95mm_HandSolder -> Capacitor_SMD:C_0603_1608Metric; LCSC C15849 -> C519554; MPN (none) -> CC0603JRX7R9BB473; Price (none) -> 0.0026
- C10, C15, C17, C2, C24, C4: value 100n -> 100nF; LCSC (none) -> C160831; MPN (none) -> CL03A104KQ3NNNC; Price (none) -> 0.0007
- C13, C18, C21, C22: value 100n -> 100nF; footprint Capacitor_SMD:C_0402_1005Metric -> Capacitor_SMD:C_0201_0603Metric; LCSC (none) -> C160831; MPN (none) -> CL03A104KQ3NNNC; Price (none) -> 0.0007
- C14, C5, C6, C7: footprint Capacitor_SMD:C_0603_1608Metric -> Capacitor_SMD:C_0201_0603Metric; LCSC C1525 -> C160831; MPN (none) -> CL03A104KQ3NNNC; Price (none) -> 0.0007
- C19: value 1u -> 1uF; footprint Capacitor_SMD:C_0402_1005Metric -> Capacitor_SMD:C_0201_0603Metric; LCSC (none) -> C160831; MPN (none) -> GRM033R60J105KEA2D; Price (none) -> 0.0007
- C2, C3: LCSC (none) -> C17024; MPN (none) -> CL21A106KPFNNNE; Price (none) -> 0.0050
- C2: value 10uF/10V (20%) -> 10uF; footprint Capacitor_SMD:C_0603_1608Metric -> Capacitor_SMD:C_0805_2012Metric; LCSC (none) -> C17024; MPN (none) -> CL21A106KPFNNNE; Price (none) -> 0.0050
- C26, C28, C30, C31, C33, C34, C8: value 1u -> 1uF; LCSC (none) -> C160831; MPN (none) -> GRM033R60J105KEA2D; Price (none) -> 0.0007
- C27: footprint Capacitor_SMD:C_0402_1005Metric -> Capacitor_SMD:C_0805_2012Metric; LCSC (none) -> C17024; MPN (none) -> CL21A106KPFNNNE; Price (none) -> 0.0050
- C29, C32: LCSC (none) -> C160831; MPN (none) -> CL03A104KQ3NNNC; Price (none) -> 0.0007
- D1, D2, D3: LCSC (none) -> C27636112; Price (none) -> 0.0092
- D10, D5, D6, D7, D8, D9: MPN B5819W SL -> B5819WT; Price (none) -> 0.0179
- J2, J4: LCSC (none) -> C566239; Price None -> 0.1080
- J3: LCSC (none) -> C3169593; Price (none) -> 1.1229
- J9: LCSC (none) -> C456013; Price (none) -> 0.2623
- L1, L10, L11, L12, L13, L2, L3, L4, L5, L6, L7, L8: Price (none) -> 0.0492
- L5: Price (none) -> 0.0208
- Q1, Q2: LCSC (none) -> C916372; MPN (none) -> MMBT2222A; Price (none) -> 0.0050
- Q4, Q5: Price (none) -> 0.037
- Q7, Q8: LCSC (none) -> C2891808; Price (none) -> 0.0035
- R1, R2, R38, R4: footprint Resistor_SMD:R_0603_1608Metric_Pad0.98x0.95mm_HandSolder -> Resistor_SMD:R_0201_0603Metric; LCSC (none) -> C106227; MPN (none) -> RC0201FR-070RL; Price (none) -> 0.0005
- R10, R11, R12, R13, R15, R16, R17, R18, R20, R23, R6, R7: LCSC (none) -> C138165; MPN (none) -> RC0201FR-071KL; Price (none) -> 0.0006
- R21, R24, R25, R26, R31, R32, R33: LCSC (none) -> C106225; MPN (none) -> RC0201FR-0710KL; Price (none) -> 0.0006
- R22: value 330 -> 330R; footprint Resistor_SMD:R_0402_1005Metric -> Resistor_SMD:R_0201_0603Metric; LCSC (none) -> C274872; MPN (none) -> RC0201FR-07330RL; Price (none) -> 0.0006
- R27, R28: value 0 -> 0R; LCSC (none) -> C106227; MPN (none) -> RC0201FR-070RL; Price (none) -> 0.0005
- R29, R30: value 27 -> 27R; LCSC (none) -> C273268; MPN (none) -> RC0201FR-0727RL; Price (none) -> 0.0006
- R3: value 100 -> 100R; LCSC (none) -> C77623; MPN (none) -> RC0201FR-07100RL; Price (none) -> 0.0006
- R3, R39: footprint Resistor_SMD:R_0402_1005Metric -> Resistor_SMD:R_0201_0603Metric; LCSC C25804 -> C106225; MPN (none) -> RC0201FR-0710KL; Price (none) -> 0.0006
- R34, R35: footprint Resistor_SMD:R_0603_1608Metric -> Resistor_SMD:R_0201_0603Metric; LCSC (none) -> C2107901; MPN (none) -> AF0201FR-0775KL; Price (none) -> 0.0006
- R37, R41: footprint Resistor_SMD:R_0402_1005Metric -> Resistor_SMD:R_0201_0603Metric; MPN (none) -> RC0201FR-070RL; Price (none) -> 0.0005
- R40, R5: footprint Resistor_SMD:R_0402_1005Metric -> Resistor_SMD:R_0201_0603Metric; LCSC C22775 -> C77623; MPN (none) -> RC0201FR-07100RL; Price (none) -> 0.0006
- R8, R9: LCSC (none) -> C274341; MPN (none) -> RC0201FR-075K1L; Price (none) -> 0.0004
- SW1: Price (none) -> 0.0458
- SW1, SW2: Price (none) -> 1.90
- SW4: LCSC (none) -> C412366; Price (none) -> 0.053
- U10, U8: LCSC (none) -> C635958; Price (none) -> 1.11
- U11, U5: Price (none) -> 0.59
- U12: Price (none) -> 0.13
- U16: Price (none) -> 1.23
- U2: Price (none) -> 0.22
- U4: LCSC (none) -> C28060; Price None -> 0.565
- U6: LCSC (none) -> C2040; Price (none) -> 0.531
- U7: Price (none) -> 0.23
- U9: LCSC (none) -> C2980306; Price (none) -> 3.18
Connections:
- net GND: now also C35.2, C36.2, Y1.2, Y1.4
- net XTAL_IN: now also C35.1, Y1.1
- net XTAL_OUT: now also R19.1
- new net: C36.1, R19.2, Y1.3

Commit message: Update production files
Parts:
- C1: Package (none) -> CASE-A-3216-18(mm)
- C10, C11, C12, C9: Package (none) -> 0603
- C10, C13, C14, C15, C17, C18, C2, C21, C22, C24, C29, C32, C4, C5, C6, C7, R1, R10, R11, R12, R13, R15, R16, R17, R18, R19, R2, R20, R21, R22, R23, R24, R25, R26, R27, R28, R29, R3, R30, R31, R32, R33, R34, R35, R38, R39, R4, R40, R5, R6, R7, R8, R9: Package (none) -> 0201
- C19, C26, C28, C30, C31, C33, C34, C8: LCSC C160831 -> C76929; Package (none) -> 0201
- C2, C27, C3: Package (none) -> 0805
- C35, C36: Package (none) -> 0402
- D1, D2, D3: Package (none) -> SOD-323
- D10, D5, D6, D7, D8, D9: Package (none) -> SOD-523
- J1: now not fitted
- J3: MPN molex_5051101492_14P -> 5051101492; Package (none) -> SMD,P=0.5mm,Surface Mount，Right Angle
- J9: Link (none) -> https://www.lcsc.com/product-detail/USB-Connectors_SHOU-HAN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; Package (none) -> -
- L1, L10, L11, L12, L13, L2, L3, L4, L5, L6, L7, L8: Link (none) -> https://cdn-shop.adafruit.com/product-files/5849/SK6805-EC1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; Package (none) -> SK6805-EC-10
- L5: Package (none) -> 1008
- Q1, Q2, Q7, Q8: Package (none) -> SOT-23
- Q4, Q5: Package (none) -> SC-70-6(SOT-363)
- R37, R41: LCSC C22775 -> C106227; Package (none) -> 0201
- SW1: Package (none) -> SMD,1.6x2.6mm
- SW1, SW2, U9: Package (none) -> -
- SW4: Package (none) -> SMD,3.3x4.5mm
- U10, U8: Package (none) -> MSOP-8
- U11, U5: Package (none) -> LGA-14(2.5x3)
- U12: Package (none) -> UQFN-10(1.5x2)
- U16: Package (none) -> DSBGA-8(1.1x1.6)
- U2: Package (none) -> USON-8-EP(2x3)
- U6: Package (none) -> LQFN-56(7x7)
- U7: Package (none) -> ESSOP-10-150mil-1mm
- Y1: Package (none) -> SMD3225-4P

Commit message: PCB Fix BOM
Parts:
- C10, C11, C12, C9: MPN CC0603JRX7R9BB473 -> TAJA476K006RNJ
Changed lines of the file:
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@@
 			)
 		)
-		(property "MPN" "CC0603JRX7R9BB473"
+		(property "MPN" "TAJA476K006RNJ"
 			(at 83.82 125.73 0)
 			(effects
@@
 			)
 		)
-		(property "MPN" "CC0603JRX7R9BB473"
+		(property "MPN" "TAJA476K006RNJ"
 			(at 95.25 100.33 0)
 			(effects
@@
 			)
 		)
-		(property "MPN" "CC0603JRX7R9BB473"
+		(property "MPN" "TAJA476K006RNJ"
 			(at 83.82 99.06 0)
 			(effects
@@
 			)
 		)
-		(property "MPN" "CC0603JRX7R9BB473"
+		(property "MPN" "TAJA476K006RNJ"
 			(at 95.25 129.54 0)
 			(effects
@@
 			)
 		)
-		(property "Description" "50mW Thick Film Resistors 25V ±1% 0Ω"
+		(property "Description" "0mW Thick Film Resistors 25V ±1% 0Ω"
 			(at 459.74 77.47 0)
 			(effects
@@
 			)
 		)
-		(property "Description" "50mW Thick Film Resistors 25V ±1% 0Ω"
+		(property "Description" "0mW Thick Film Resistors 25V ±1% 0Ω"
 			(at 459.74 25.4 0)
 			(effects
