File: PCB/main_3.3/progcc_3.3_main.kicad_pcb (KiCad board)
At the start: 4 copper layers, 110.9 x 59.7 mm, 124 parts, among them J1 Conn_01x04_Pin, J2 SM02B-SURS-TF_LF__SN_, J3 To Button Board, J4 SM02B-SURS-TF_LF__SN_, J5 Conn_01x02_Pin, J9 USB_C_Receptacle, P1 RPI-RM2, Q1 MMBT2222A, Q2 MMBT2222A, Q4 BSS138DW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

Commit message: Routing
Parts:
- D1, D2, D3, D4: value CUS08F30 -> CUS08F30,H3F
- L14: value L -> BLM18AG601SN1D
- moved R1 60.5 mm to (137.6, 140.8)
- moved R2 58.0 mm to (143.8, 133.2)
- moved L14 51.9 mm to (143.7, 126.4), turned to -90 degrees
- moved C7 32.6 mm to (113.0, 111.1), turned to 180 degrees
- moved R24 26.2 mm to (118.5, 115.4), turned to 90 degrees
- moved S1 25.8 mm to (115.9, 122.0)
- moved C37 25.3 mm to (114.5, 125.3), turned to -90 degrees
- moved R25 24.0 mm to (118.5, 113.9), turned to 90 degrees
- moved R23 18.6 mm to (148.6, 112.4), turned to -90 degrees
- moved R20 17.6 mm to (147.8, 111.1), turned to -90 degrees
- moved C5 7.59 mm to (115.2, 119.1)
- moved C6 6.39 mm to (118.9, 118.0), turned to 90 degrees
- moved D4 1.59 mm to (149.4, 114.0)
- moved U11 0.78 mm to (115.2, 113.0)
- moved U5 0.78 mm to (115.7, 117.0)
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Connections:
- S1 pad 2: LX -> LY
- S1 pad 4: LY -> LX
Routing:
- net I2C1_SCL: track 0.00 -> 39.4 mm, vias 0 -> 4
- net ADC_MUX_OUT: track 0.00 -> 39.0 mm, vias 0 -> 2
- net RY: track 34.8 -> 72.9 mm, vias 2 -> 4
- net RX: track 35.2 -> 72.9 mm, vias 2 -> 4
- net ADC_ADDR_1: track 2.90 -> 32.6 mm, vias 1 -> 2
- net ADC_ADDR_0: track 0.00 -> 28.7 mm, vias 0 -> 2
- net WL_CLK: track 11.6 -> 35.6 mm, vias 1 -> 2
- net +3V3: track 82.6 -> 106.4 mm, vias 31 -> 36
- net GND: track 61.8 -> 82.5 mm, vias 48 -> 56
- net UART0_TX: track 5.78 -> 25.1 mm, vias 0 -> 1
- net I2C1_SDA: track 18.2 -> 34.0 mm
- net RGB_OUT: track 36.7 -> 20.9 mm
- net WL_CS: track 12.3 -> 26.0 mm, vias 1 -> 0
- net MODE_BUTTON: track 28.1 -> 14.9 mm, vias 3 -> 2
- net (no net): track 16.3 -> 3.80 mm
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Other:
- board text added: "Design by Mitch Cairns 2.4.2025"
- board text added: "ProGCC 3.3"
- board text removed: "Design by Mitch Cairns 10.26.2024"
- board text removed: "ProGCC 3.2"

Commit message: Safety
Parts:
- added U1: USBLC6-2P6, Package_TO_SOT_SMD:SOT-666, F.Cu at (138.6, 103.6)
- added U2: USBLC6-2P6, Package_TO_SOT_SMD:SOT-666, F.Cu at (133.8, 102.8)
- added U3: USBLC6-2P6, Package_TO_SOT_SMD:SOT-666, F.Cu at (136.3, 102.8)
- moved R9 2.89 mm to (132.2, 101.2)
- moved C1 1.44 mm to (133.9, 105.5), turned to 180 degrees
Connections:
- Q4 pad 4: N_LATCH -> N_LATCH_SAFE
- Q5 pad 4: N_DATA -> N_DATA_SAFE
- Q5 pad 6: N_CLOCK -> N_CLOCK_SAFE
- R11 pad 2: N_LATCH -> N_LATCH_SAFE
- R12 pad 2: N_CLOCK -> N_CLOCK_SAFE
- R13 pad 2: N_DATA -> N_DATA_SAFE
- R29 pad 1: D+ -> SAFE_D+
- R30 pad 1: D- -> SAFE_D-
- TP1 pad 1: N_LATCH -> N_LATCH_SAFE
- TP2 pad 1: N_CLOCK -> N_CLOCK_SAFE
- TP3 pad 1: N_DATA -> N_DATA_SAFE
Routing:
- net N_DATA: track 32.6 -> 11.7 mm, vias 4 -> 1
- net N_LATCH: track 33.6 -> 13.0 mm
- net N_LATCH_SAFE: track 0.00 -> 17.4 mm, vias 0 -> 1
- net N_CLOCK: track 32.4 -> 15.2 mm, vias 4 -> 2
- net N_CLOCK_SAFE: track 0.00 -> 16.3 mm, vias 0 -> 2
- net N_DATA_SAFE: track 0.00 -> 15.8 mm, vias 0 -> 2
- net D+: track 30.7 -> 23.6 mm
- net D-: track 30.0 -> 23.0 mm
- net VBUS_PRE: track 26.2 -> 31.8 mm, vias 3 -> 4
- net SAFE_D+: track 0.00 -> 5.17 mm
- net SAFE_D-: track 0.00 -> 4.60 mm
- net GND: track 82.5 -> 86.9 mm
- net /CC2: track 13.1 -> 10.1 mm
- net +3.3V_PRE: track 33.0 -> 33.8 mm, vias 1 -> 2

Commit message: V3.3
Routing:
- net GND: track 86.9 -> 88.4 mm

Commit message: V3S
Parts:
- added TP5: TestPoint, TestPoint:TestPoint_Pad_2.5x2.5mm, B.Cu at (133.6, 116.2)
- added TP6: TestPoint, TestPoint:TestPoint_Pad_2.5x2.5mm, B.Cu at (133.6, 119.7)
- moved C20 4.07 mm to (158.2, 112.3)
- moved C23 3.59 mm to (161.2, 117.9)
- moved L9 3.59 mm to (162.0, 111.8)
- moved R36 3.59 mm to (160.5, 118.7)
- moved U14 3.59 mm to (161.3, 115.5)
- moved REF** 3.42 mm to (159.0, 123.4)
- moved C25 1.60 mm to (165.1, 112.2), turned to 90 degrees
Routing:
- net /SWD: track 0.00 -> 10.7 mm, vias 0 -> 1
- net /SWCLK: track 0.00 -> 9.65 mm, vias 0 -> 1
- net GND: track 88.4 -> 84.7 mm, vias 56 -> 55
- net VBUS_SYS: track 30.8 -> 34.2 mm
- net Push_A: track 56.6 -> 54.1 mm
- net Scan_C: track 55.9 -> 53.4 mm
- net Scan_B: track 53.7 -> 51.2 mm
- net Push_C: track 53.1 -> 50.6 mm
- net Push_D: track 54.6 -> 52.1 mm
- net Scan_A: track 54.5 -> 52.1 mm
- net Push_B: track 55.1 -> 52.6 mm
- net Scan_D: track 54.4 -> 51.9 mm
- net +3V3: track 106.5 -> 108.3 mm
- net BAT_LVL: track 85.8 -> 86.5 mm
Other:
- board text added: "Design by Mitch Cairns 7.14.2025"
- board text removed: "Design by Mitch Cairns 2.4.2025"
