File: PCB/main_3.3/progcc_3.3_main.kicad_sch (KiCad schematic)
At the start: 123 parts, among them J1 Conn_01x04_Pin, J2 SM02B-SURS-TF_LF__SN_, J3 To Button Board, J4 SM02B-SURS-TF_LF__SN_, J5 Conn_01x02_Pin, J9 USB_C_Receptacle, P1 RPI-RM2, Q1 MMBT2222A, Q2 MMBT2222A, Q4 BSS138DW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

Commit message: Routing
Parts:
- D1, D2, D3: value CUS08F30 -> CUS08F30,H3F; LCSC C27636112 -> C150183; MPN CUS08F30 -> CUS08F30,H3F
- L14: value L -> BLM18AG601SN1D; LCSC (none) -> C19330; MPN (none) -> BLM18AG601SN1D; Package (none) -> 0603
- R1: LCSC (none) -> C226558; MPN (none) -> AC0201FR-07470RL
Connections:
- net LX: now also S1.4 (S3); no longer S1.2 (S1)
- net LY: now also S1.2 (S1); no longer S1.4 (S3)
Other:
- moved on the sheet: C37, S1

Commit message: Safety
Parts:
- added U1, U2, U3: USBLC6-2P6, Package_TO_SOT_SMD:SOT-666, symbol Power_Protection:USBLC6-2P6
Connections:
- net +3.3V_PRE: now also U3.5 (VBUS)
- net D+: now also U1.3 (I/O2); no longer R29.1
- net D-: now also U1.1 (I/O1); no longer R30.1
- net GND: now also U1.2 (GND), U2.2 (GND), U3.2 (GND)
- net N_CLOCK: now also U2.4 (I/O2); no longer Q5.6 (D1), R12.2, TP2.1
- net N_DATA: now also U3.6 (I/O1); no longer Q5.4 (S2), R13.2, TP3.1
- net N_LATCH: now also U2.6 (I/O1); no longer Q4.4 (S2), R11.2, TP1.1
- net VBUS_PRE: now also U1.5 (VBUS)
- new net N_CLOCK_SAFE: Q5.6 (D1), R12.2, TP2.1, U2.3 (I/O2)
- new net N_DATA_SAFE: Q5.4 (S2), R13.2, TP3.1, U3.1 (I/O1)
- new net N_LATCH_SAFE: Q4.4 (S2), R11.2, TP1.1, U2.1 (I/O1)
- new net SAFE_D+: R29.1, U1.4 (I/O2)
- new net SAFE_D-: R30.1, U1.6 (I/O1)
Other:
- note added: "ESD"

Commit message: V3.3
Parts:
- L14, R1, R2: USBDNP (none) -> YES
- P1: MPN (none) -> RPI-RM2; USBDNP (none) -> YES
- U1, U2, U3: LCSC (none) -> C2827693; MPN (none) -> USBLC6-2P6; Package (none) -> SOT-666-6
Other:
- note added: "Analog Mux"
- note added: "Haptics Driver L"
- note added: "Haptics Driver R"
- note added: "Haptics Output"
- note added: "RPI-RM2 Wireless"
- note removed: "Haptics"
- note removed: "Rumble"
- moved on the sheet: C1, C10, C11, C12, C13, C14, C17, C18, C19, C2, C21, C22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

Commit message: V3S
Parts:
- added TP5, TP6: TestPoint, TestPoint:TestPoint_Pad_2.5x2.5mm, symbol Connector:TestPoint
Connections:
- net SWCLK: now also TP5.1
- net SWD: now also TP6.1
Other:
- title: ProGCC 3.2 Main Board -> ProGCC 3.3 Main Board
Changed lines of the file:
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@@
 	(paper "User" 465 350)
 	(title_block
-		(title "ProGCC 3.2 Main Board")
+		(title "ProGCC 3.3 Main Board")
 		(date "2019-12-18")
 		(rev "0.1")
@@
 	)
 	(symbol
+		(lib_id "Connector:TestPoint")
+		(at 364.49 168.91 90)
+		(unit 1)
+		(exclude_from_sim no)
+		(in_bom yes)
+		(on_board yes)
+		(dnp no)
+		(property "Reference" "TP6"
+			(at 358.394 168.91 90)
+			(effects
+				(font
+					(size 1.27 1.27)
+				)
+			)
+		)
+		(property "Value" "TestPoint"
+			(at 361.188 171.45 90)
+			(effects
+				(font
+					(size 1.27 1.27)
+				)
+				(hide yes)
+			)
+		)
+		(property "Footprint" "TestPoint:TestPoint_Pad_2.5x2.5mm"
+			(at 364.49 163.83 0)
+			(effects
+				(font
+					(size 1.27 1.27)
+				)
+				(hide yes)
+			)
+		)
+		(property "Datasheet" "~"
+			(at 364.49 163.83 0)
+			(effects
+				(font
+					(size 1.27 1.27)
+				)
+				(hide yes)
+			)
+		)
+		(property "Description" "test point"
+			(at 364.49 168.91 0)
+			(effects
+				(font
+					(size 1.27 1.27)
+				)
+				(hide yes)
+			)
+		)
+		(pin "1"
+		)
+		(instances
+			(project "progcc_3.3_main"
+				(path "/9ec9c1c0-f5f6-4920-ad47-c5d4aa989114"
+					(reference "TP6")
+					(unit 1)
+				)
+			)
+		)
+	)
+	(symbol
 		(lib_id "power:+3V3")
 		(at 93.98 203.2 90)
@@
 					(unit 1)
 				)
+			)
+		)
+	)
+	(symbol
+		(lib_id "Connector:TestPoint")
+		(at 364.49 166.37 90)
+		(unit 1)
+		(exclude_from_sim no)
+		(in_bom yes)
+		(on_board yes)
+		(dnp no)
+		(property "Reference" "TP5"
+			(at 358.394 166.624 90)
+			(effects
+				(font
+					(size 1.27 1.27)
+				)
+			)
+		)
+		(property "Value" "TestPoint"
+			(at 358.648 164.084 90)
+			(effects
+				(font
+					(size 1.27 1.27)
+				)
+				(hide yes)
+			)
+		)
+		(property "Footprint" "TestPoint:TestPoint_Pad_2.5x2.5mm"
+			(at 364.49 161.29 0)
+			(effects
+				(font
+					(size 1.27 1.27)
+				)
+				(hide yes)
+			)
+		)
+		(property "Datasheet" "~"
+			(at 364.49 161.29 0)
+			(effects
+				(font
+					(size 1.27 1.27)
+				)
+				(hide yes)
+			)
+		)
+		(property "Description" "test point"
+			(at 364.49 166.37 0)
+			(effects
+				(font
+					(size 1.27 1.27)
+				)
+				(hide yes)
+			)
+		)
+		(pin "1"
+		)
+		(instances
+			(project "progcc_3.3_main"
+				(path "/9ec9c1c0-f5f6-4920-ad47-c5d4aa989114"
+					(reference "TP5")
+					(unit 1)
+				)
