File: PCB/main_3S/progcc_3S_main.kicad_sch (KiCad schematic)
At the start: 113 parts, among them J1 USB4056-03-A, J2 To Button Board, J3 USB_C_Receptacle, J4 SM02B-SURS-TF_LF__SN_, J5 SM02B-SURS-TF_LF__SN_, J6 Conn_01x02_Pin, Q1 MMBT2222A, Q2 MMBT2222A, Q3 BSS138DW, Q4 BSS138DW, SW1 GL1807SYAE-002, SW2 GL1807SYAE-002, SW3 TS35CA, SW4 1TS026A-1000-0550, T1 36-8730, T2 36-8730, T3 36-8730, T4 36-8730, U1 USBLC6-2P6, U2 USBLC6-2P6, U3 USBLC6-2P6, U4 ST_LSM6, U5 ST_LSM6, U6 TPS63001DRCR, U7 RP2350_60QFN, Y1 ABM8-272-T3

Commit message: 3S Resistor Update
Parts:
- C10, C11, C7, C8: MPN TAJA476K006RNJ -> CC0603JRX7R9BB473
- C9: MPN CC0603JRX7R9BB473 -> TAJA476K006RNJ
- R31: value 100R -> 27R; LCSC C77623 -> C273268; MPN RC0201FR-07100RL -> RC0201FR-0727RL
